File: hardware/waagen/elektronik/kiCAD/CAN.kicad_sch (KiCad schematic)
At the start: 8 parts, among them U3 SN65HVD230, U4 MCP2515, Y2 8MHz

Commit message: Error on JP1 fixed and changed scale wires pads
Parts:
- Y2: footprint Crystal:Crystal_SMD_HC49-SD -> Crystal:Crystal_SMD_HC49-SD_HandSoldering
Changed lines of the file:
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@@
       (effects (font (size 1.27 1.27)) (justify right))
     )
-    (property "Footprint" "Crystal:Crystal_SMD_HC49-SD" (id 2) (at 121.92 111.76 0)
+    (property "Footprint" "Crystal:Crystal_SMD_HC49-SD_HandSoldering" (id 2) (at 121.92 111.76 0)
       (effects (font (size 1.27 1.27)) hide)
     )
