File: hardware/waagen/elektronik/kiCAD/scale.kicad_sch (KiCad schematic)
At the start: 12 parts, among them J4 Conn_01x03_Male, J5 Conn_01x03_Male, J7 Conn_01x03_Male, J8 Conn_01x03_Male, U5 NAU7802SGI

Commit message: Error on JP1 fixed and changed scale wires pads
Parts:
- J4, J5, J7, J8: footprint Connector_PinHeader_2.54mm:PinHeader_1x03_P2.54mm_Vertical -> Connector_Wire:SolderWire-0.1sqmm_1x03_P3.6mm_D0.4mm_OD1mm_Relief2x
Changed lines of the file:
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@@
     (property "Reference" "J7" (id 0) (at 113.665 60.96 0))
     (property "Value" "Conn_01x03_Male" (id 1) (at 113.665 63.5 0))
-    (property "Footprint" "Connector_PinHeader_2.54mm:PinHeader_1x03_P2.54mm_Vertical" (id 2) (at 113.03 68.58 0)
+    (property "Footprint" "Connector_Wire:SolderWire-0.1sqmm_1x03_P3.6mm_D0.4mm_OD1mm_Relief2x" (id 2) (at 113.03 68.58 0)
       (effects (font (size 1.27 1.27)) hide)
     )
@@
     (property "Reference" "J5" (id 0) (at 89.535 60.96 0))
     (property "Value" "Conn_01x03_Male" (id 1) (at 89.535 63.5 0))
-    (property "Footprint" "Connector_PinHeader_2.54mm:PinHeader_1x03_P2.54mm_Vertical" (id 2) (at 88.9 68.58 0)
+    (property "Footprint" "Connector_Wire:SolderWire-0.1sqmm_1x03_P3.6mm_D0.4mm_OD1mm_Relief2x" (id 2) (at 88.9 68.58 0)
       (effects (font (size 1.27 1.27)) hide)
     )
@@
     (property "Reference" "J8" (id 0) (at 139.065 60.96 0))
     (property "Value" "Conn_01x03_Male" (id 1) (at 139.065 63.5 0))
-    (property "Footprint" "Connector_PinHeader_2.54mm:PinHeader_1x03_P2.54mm_Vertical" (id 2) (at 138.43 68.58 0)
+    (property "Footprint" "Connector_Wire:SolderWire-0.1sqmm_1x03_P3.6mm_D0.4mm_OD1mm_Relief2x" (id 2) (at 138.43 68.58 0)
       (effects (font (size 1.27 1.27)) hide)
     )
@@
     (property "Reference" "J4" (id 0) (at 64.135 60.96 0))
     (property "Value" "Conn_01x03_Male" (id 1) (at 64.135 63.5 0))
-    (property "Footprint" "Connector_PinHeader_2.54mm:PinHeader_1x03_P2.54mm_Vertical" (id 2) (at 63.5 68.58 0)
+    (property "Footprint" "Connector_Wire:SolderWire-0.1sqmm_1x03_P3.6mm_D0.4mm_OD1mm_Relief2x" (id 2) (at 63.5 68.58 0)
       (effects (font (size 1.27 1.27)) hide)
     )
