File: hardware/waagen/waage_v4/elektronik/Untitled.kicad_sch (KiCad schematic)
At the start: 9 parts, among them J1 USB_A, J2 Conn_01x03, J3 USB_A, SW1 SW_Push, U1 ATtiny414-SS

Commit message: intermediate step
Parts:
- removed J1: USB_A, Library_USB_A:Conn_USB_A_Jack, symbol Connector:USB_A
- removed J3: USB_A, Library_USB_A:Conn_USB_A_Plug, symbol Connector:USB_A
- removed SW1: SW_Push, Library_USB_A:Button_Switch_ESE-11MV1T, symbol Switch:SW_Push
- removed U1: ATtiny414-SS, Package_SO:SOIC-14_3.9x8.7mm_P1.27mm, symbol MCU_Microchip_ATtiny:ATtiny414-SS
- added J2, J3: SM04B-SRSS-TB(LF)(SN), Quiicconnector:JST_SM04B-SRSS-TB(LF)(SN), symbol connector:SM04B-SRSS-TB(LF)(SN)
- added R1: 180, Resistor_SMD:R_1206_3216Metric_Pad1.30x1.75mm_HandSolder, symbol Device:R
- added U1: ATtiny1614-SS, Package_SO:SOIC-14_3.9x8.7mm_P1.27mm, symbol MCU_Microchip_ATtiny:ATtiny1614-SS
- D1: footprint LED_THT:LED_D5.0mm_Horizontal_O3.81mm_Z9.0mm -> LED_SMD:LED_1206_3216Metric_Pad1.42x1.75mm_HandSolder
- renumbered J2 to J1
Connections:
- net GND: now also J2.1, J2.S1 (SHIELD), J2.S2 (SHIELD), J3.1, J3.S1 (SHIELD), J3.S2 (SHIELD), R1.2, U1.14 (GND); no longer D1.1 (K)
- net VCC: now also J2.2, J3.2, U1.1 (VCC)
- net at J1.2 (Pin_2): now also U1.10 (~{RESET}/PA0)
- net at D1.2 (A): now also U1.5 (PA7)
- new net: D1.1 (K), R1.1
- new net SCL_0: U1.9 (PB0)
- new net SCL_1: J2.4, J3.4, U1.12 (PA2)
- new net SDA_0: U1.8 (PB1)
- new net SDA_1: J2.3, J3.3, U1.11 (PA1)
- no-connect marks 7 -> 6
Other:
- added sheet Scale (scale2.kicad_sch)
- moved on the sheet: C1, D1, J1

Commit message: Zwischenstand Elektronik v4
Parts:
- removed H1, H2: MountingHole, MountingHole:MountingHole_2.5mm, symbol Mechanical:MountingHole
Changed lines of the file:
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@@
-    )
-  )
-  (symbol (lib_id "Mechanical:MountingHole") (at 83.82 48.26 0) (unit 1)
-    (in_bom yes) (on_board yes) (dnp no) (fields_autoplaced)
-    (property "Reference" "H2" (at 86.36 46.9899 0)
-      (effects (font (size 1.27 1.27)) (justify left))
-    )
-    (property "Value" "MountingHole" (at 86.36 49.5299 0)
-      (effects (font (size 1.27 1.27)) (justify left))
-    )
-    (property "Footprint" "MountingHole:MountingHole_2.5mm" (at 83.82 48.26 0)
-      (effects (font (size 1.27 1.27)) hide)
-    )
-    (property "Datasheet" "~" (at 83.82 48.26 0)
-      (effects (font (size 1.27 1.27)) hide)
-    )
-    (instances
-      (project "Untitled"
-        (path "/e63e39d7-6ac0-4ffd-8aa3-1841a4541b55"
-          (reference "H2") (unit 1)
-        )
-      )
-    )
-  )
-  (symbol (lib_id "Mechanical:MountingHole") (at 83.82 43.18 0) (unit 1)
-    (in_bom yes) (on_board yes) (dnp no) (fields_autoplaced)
-    (property "Reference" "H1" (at 86.36 41.9099 0)
-      (effects (font (size 1.27 1.27)) (justify left))
-    )
-    (property "Value" "MountingHole" (at 86.36 44.4499 0)
-      (effects (font (size 1.27 1.27)) (justify left))
-    )
-    (property "Footprint" "MountingHole:MountingHole_2.5mm" (at 83.82 43.18 0)
-      (effects (font (size 1.27 1.27)) hide)
-    )
-    (property "Datasheet" "~" (at 83.82 43.18 0)
-      (effects (font (size 1.27 1.27)) hide)
-    )
-    (instances
-      (project "Untitled"
-        (path "/e63e39d7-6ac0-4ffd-8aa3-1841a4541b55"
-          (reference "H1") (unit 1)
-        )
-      )
     )
   )

Commit message: Datein für die Produktion
Other:
- note added: "PA6 - do not use. used for interenal chip tests"
Changed lines of the file:
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@@
     (stroke (width 0) (type default))
+  )
+  (text "PA6 - do not use. used for interenal chip tests" (at 123.19 92.71 0)
+    (effects (font (size 1.27 1.27)) (justify left bottom))
   )
   (label "SDA_0" (at 82.55 78.74 0) (fields_autoplaced)
